File: PCB/SolderDispenser v1.1.brd (EAGLE design)
At the start: 39 x 95 mm, 44 parts, among them IC1 ULN2003AD, U2 ATMEGA328P_TQFP

Commit message: add missing crystal value
Parts:
- Q1: value (none) -> 12Mhz
- Q2: value (none) -> 16Mhz
Changed lines of the file:
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@@
 <?xml version="1.0" encoding="utf-8"?>
 <!DOCTYPE eagle SYSTEM "eagle.dtd">
-<eagle version="9.6.1">
+<eagle version="9.6.2">
 <drawing>
 <settings>
@@
 <attribute name="VALUE" x="19.584" y="-43.451" size="0.4064" layer="27" ratio="10"/>
 </element>
-<element name="Q1" library="adafruit" library_urn="urn:adsk.eagle:library:420" package="HC49UP" package3d_urn="urn:adsk.eagle:package:6240908/1" value="" x="24.69" y="26.72" smashed="yes" rot="R180">
+<element name="Q1" library="adafruit" library_urn="urn:adsk.eagle:library:420" package="HC49UP" package3d_urn="urn:adsk.eagle:package:6240908/1" value="12Mhz" x="24.69" y="26.72" smashed="yes" rot="R180">
 <attribute name="MF" value="" x="-22.3" y="44.5" size="1.778" layer="27" rot="R180" display="off"/>
 <attribute name="MPN" value="" x="-22.3" y="44.5" size="1.778" layer="27" rot="R180" display="off"/>
@@
 <attribute name="VALUE" x="30.405" y="30.911" size="1.27" layer="27" ratio="10" rot="R180"/>
 </element>
-<element name="Q2" library="adafruit" library_urn="urn:adsk.eagle:library:420" package="HC49UP" package3d_urn="urn:adsk.eagle:package:6240908/1" value="" x="9.77" y="8.62" smashed="yes" rot="R270">
+<element name="Q2" library="adafruit" library_urn="urn:adsk.eagle:library:420" package="HC49UP" package3d_urn="urn:adsk.eagle:package:6240908/1" value="16Mhz" x="9.77" y="8.62" smashed="yes" rot="R270">
 <attribute name="MF" value="" x="-16.9" y="-11.7" size="1.778" layer="27" rot="R270" display="off"/>
 <attribute name="MPN" value="" x="-16.9" y="-11.7" size="1.778" layer="27" rot="R270" display="off"/>
